Commit message: mejora de algoritmo de identificacion de objetos, 2 puntos extremos y el mas cercano

File: roverbot_description/urdf/roverbot.xacro (robot description, xacro)
@@ -102,14 +102,14 @@
 	<!-- Roverbot wheel macros -->
 	<xacro:roverbotWheel wheel="rightBackTire" axle="backAxle">
-		<origin xyz="${WheelPositionX} ${-WheelPositionY} ${WheelPositionZ}"/>
+		<origin rpy="-1.5708 0 0" xyz="${WheelPositionX} ${-WheelPositionY} ${WheelPositionZ}"/>
 	</xacro:roverbotWheel>
 	<xacro:roverbotWheel wheel="leftBackTire" axle="backAxle">
-		<origin xyz="${WheelPositionX} ${WheelPositionY} ${WheelPositionZ}"/>
+		<origin rpy="-1.5708 0 0" xyz="${WheelPositionX} ${WheelPositionY} ${WheelPositionZ}"/>
 	</xacro:roverbotWheel>
 	<xacro:roverbotWheel wheel="rightFrontTire" axle="frontAxle">
-		<origin xyz="${WheelPositionX} ${-WheelPositionY} ${WheelPositionZ}"/>
+		<origin rpy="-1.5708 0 0" xyz="${WheelPositionX} ${-WheelPositionY} ${WheelPositionZ}"/>
 	</xacro:roverbotWheel>
 	<xacro:roverbotWheel wheel="leftFrontTire" axle="frontAxle">
-		<origin xyz="${WheelPositionX} ${WheelPositionY} ${WheelPositionZ}"/>
+		<origin rpy="-1.5708 0 0" xyz="${WheelPositionX} ${WheelPositionY} ${WheelPositionZ}"/>
 	</xacro:roverbotWheel>
 	<!--Bumpers-->

File: roverbot_description/urdf/roverbotWheel.xacro (robot description, xacro)
@@ -10,5 +10,5 @@
 			</inertial>
 			<visual>
-				<origin xyz="0 0 0" rpy="0 0 0" />
+				<origin xyz="0 0 0" rpy="${PI/2} 0 0" />
 				<geometry>
 					<!--cylinder length="${wheelLength}" radius="${wheelRadius}" /-->
@@ -17,5 +17,4 @@
 			</visual>
 			<collision>
-				<origin xyz="0 0 0" rpy="${PI/2} 0 0" />
 				<geometry>
 					<cylinder length="${wheelLength}" radius="${wheelRadius}" />
@@ -34,5 +33,5 @@
 			<child link="${wheel}"/>
 			<xacro:insert_block name="joint_pose"/>
-			<axis xyz="0 1 0" rpy="0 0 0" />
+			<axis xyz="0 0 1" />
 		</joint>
 	</xacro:macro>

Commit message: Arreglada movimiento del robot

File: roverbot_description/urdf/roverbot.xacro (robot description, xacro)
@@ -102,14 +102,14 @@
 	<!-- Roverbot wheel macros -->
 	<xacro:roverbotWheel wheel="rightBackTire" axle="backAxle">
-		<origin rpy="-1.5708 0 0" xyz="${WheelPositionX} ${-WheelPositionY} ${WheelPositionZ}"/>
+		<origin rpy="${-PI/2} 0 0" xyz="${WheelPositionX} ${-WheelPositionY} ${WheelPositionZ}"/>
 	</xacro:roverbotWheel>
 	<xacro:roverbotWheel wheel="leftBackTire" axle="backAxle">
-		<origin rpy="-1.5708 0 0" xyz="${WheelPositionX} ${WheelPositionY} ${WheelPositionZ}"/>
+		<origin rpy="${-PI/2} 0 0" xyz="${WheelPositionX} ${WheelPositionY} ${WheelPositionZ}"/>
 	</xacro:roverbotWheel>
 	<xacro:roverbotWheel wheel="rightFrontTire" axle="frontAxle">
-		<origin rpy="-1.5708 0 0" xyz="${WheelPositionX} ${-WheelPositionY} ${WheelPositionZ}"/>
+		<origin rpy="${-PI/2} 0 0" xyz="${WheelPositionX} ${-WheelPositionY} ${WheelPositionZ}"/>
 	</xacro:roverbotWheel>
 	<xacro:roverbotWheel wheel="leftFrontTire" axle="frontAxle">
-		<origin rpy="-1.5708 0 0" xyz="${WheelPositionX} ${WheelPositionY} ${WheelPositionZ}"/>
+		<origin rpy="${-PI/2} 0 0" xyz="${WheelPositionX} ${WheelPositionY} ${WheelPositionZ}"/>
 	</xacro:roverbotWheel>
 	<!--Bumpers-->
